File: KiCadProject/v1.55/PongClock.kicad_pcb (KiCad board)
At the start: 2 copper layers, 69.9 x 88.9 mm, 24 parts, among them J1 CONN_01X01_MALE, J2 MY_USB_OTG, SW1 SW_DIP_x02, SW2 SW_DIP_x02, U1 TinyRTC_I2C_RIGHT, U2 MAX7219_IN, U3 MAX7219_IN, U4 MAX7219_IN, U5 MAX7219_IN, U6 MAX7219_IN, U7 MAX7219_IN, U8 ATMEGA328P-PU, U9 FTDI1232, Y1 Crystal

Commit message: v1.55
Parts:
- moved U9 3.81 mm to (170.2, 97.8)
Connections:
- U2 pad 2: GND -> (no net)
- U3 pad 2: GND -> (no net)
- U7 pad 2: GND -> (no net)
Routing:
- net GND: track 335.8 -> 285.9 mm
- net VCC: track 271.1 -> 265.9 mm, vias 0 -> 2
- net TX: track 23.0 -> 18.1 mm
- net Net-(C3-Pad2): track 30.0 -> 25.4 mm
- net RX: track 19.4 -> 14.8 mm
- removed copper zone on F.Cu, net GND
Other:
- board size 69.9 x 88.9 mm -> 67.3 x 88.9 mm
