File: KiCadProject/v1.55/PongClock.sch (KiCad schematic (older format))
At the start: 24 parts, among them J1 CONN_01X01_MALE, J2 MY_USB_OTG, SW1 SW_DIP_x02, SW2 SW_DIP_x02, U1 TinyRTC_I2C_RIGHT, U2 MAX7219_IN, U3 MAX7219_IN, U4 MAX7219_IN, U5 MAX7219_IN, U6 MAX7219_IN, U7 MAX7219_IN, U8 ATMEGA328P-PU, U9 FTDI1232, Y1 Crystal

Commit message: v1.55
Connections:
- net GND: no longer U2.2 (GND), U3.2 (GND), U7.2 (GND)
- no-connect marks 36 -> 39
Changed lines of the file:
@@
 	0    -1   -1   0
-$EndComp
-$Comp
-L GND #PWR02
-U 1 1 596A30EB
-P 6800 4500
-F 0 "#PWR02" H 6800 4250 50  0001 C CNN
-F 1 "GND" V 6800 4300 50  0000 C CNN
-F 2 "" H 6800 4500 50  0001 C CNN
-F 3 "" H 6800 4500 50  0001 C CNN
-	1    6800 4500
-	0    1    1    0
 $EndComp
 NoConn ~ 6800 4600
@@
 $EndComp
 $Comp
-L VCC #PWR03
+L VCC #PWR02
 U 1 1 597B8E7E
 P 9050 5600
-F 0 "#PWR03" H 9050 5450 50  0001 C CNN
+F 0 "#PWR02" H 9050 5450 50  0001 C CNN
 F 1 "VCC" V 9050 5800 50  0000 C CNN
 F 2 "" H 9050 5600 50  0001 C CNN
@@
 $EndComp
 $Comp
-L GND #PWR04
+L GND #PWR03
 U 1 1 597B8E84
 P 6800 5700
-F 0 "#PWR04" H 6800 5450 50  0001 C CNN
+F 0 "#PWR03" H 6800 5450 50  0001 C CNN
 F 1 "GND" V 6800 5500 50  0000 C CNN
 F 2 "" H 6800 5700 50  0001 C CNN
@@
 NoConn ~ 6800 4800
 $Comp
-L VCC #PWR05
+L VCC #PWR04
 U 1 1 597C7538
 P 6800 5000
-F 0 "#PWR05" H 6800 4850 50  0001 C CNN
+F 0 "#PWR04" H 6800 4850 50  0001 C CNN
 F 1 "VCC" V 6800 5200 50  0000 C CNN
 F 2 "" H 6800 5000 50  0001 C CNN
@@
 $EndComp
 $Comp
-L GND #PWR06
+L GND #PWR05
 U 1 1 597C7588
 P 9050 5100
-F 0 "#PWR06" H 9050 4850 50  0001 C CNN
+F 0 "#PWR05" H 9050 4850 50  0001 C CNN
 F 1 "GND" V 9050 4900 50  0000 C CNN
 F 2 "" H 9050 5100 50  0001 C CNN
@@
 $EndComp
 $Comp
-L GND #PWR07
+L GND #PWR06
 U 1 1 598DFC0D
 P 1050 3300
-F 0 "#PWR07" H 1050 3050 50  0001 C CNN
+F 0 "#PWR06" H 1050 3050 50  0001 C CNN
 F 1 "GND" V 1050 3100 50  0000 C CNN
 F 2 "" H 1050 3300 50  0001 C CNN
@@
 $EndComp
 $Comp
-L VCC #PWR08
+L VCC #PWR07
 U 1 1 598DFC7E
 P 1050 1350
-F 0 "#PWR08" H 1050 1200 50  0001 C CNN
+F 0 "#PWR07" H 1050 1200 50  0001 C CNN
 F 1 "VCC" V 1050 1550 50  0000 C CNN
 F 2 "" H 1050 1350 50  0001 C CNN
@@
 OSC1
 $Comp
-L GND #PWR09
+L GND #PWR08
 U 1 1 598E0208
 P 4300 1500
-F 0 "#PWR09" H 4300 1250 50  0001 C CNN
+F 0 "#PWR08" H 4300 1250 50  0001 C CNN
 F 1 "GND" V 4300 1300 50  0000 C CNN
 F 2 "" H 4300 1500 50  0001 C CNN
@@
 $EndComp
 $Comp
-L GND #PWR010
+L GND #PWR09
 U 1 1 598E32E5
 P 4150 3050
-F 0 "#PWR010" H 4150 2800 50  0001 C CNN
+F 0 "#PWR09" H 4150 2800 50  0001 C CNN
 F 1 "GND" V 4150 2850 50  0000 C CNN
 F 2 "" H 4150 3050 50  0001 C CNN
@@
 $EndComp
 $Comp
-L VCC #PWR011
+L VCC #PWR010
 U 1 1 598E33DE
 P 4150 2750
-F 0 "#PWR011" H 4150 2600 50  0001 C CNN
+F 0 "#PWR010" H 4150 2600 50  0001 C CNN
 F 1 "VCC" V 4150 2950 50  0000 C CNN
 F 2 "" H 4150 2750 50  0001 C CNN
@@
 SW2
 $Comp
-L GND #PWR012
+L GND #PWR011
 U 1 1 598EBAEB
 P 4250 4600
-F 0 "#PWR012" H 4250 4350 50  0001 C CNN
+F 0 "#PWR011" H 4250 4350 50  0001 C CNN
 F 1 "GND" V 4250 4400 50  0000 C CNN
 F 2 "" H 4250 4600 50  0001 C CNN
@@
 $EndComp
 $Comp
-L VCC #PWR013
+L VCC #PWR012
 U 1 1 598EBB74
 P 4550 4000
-F 0 "#PWR013" H 4550 3850 50  0001 C CNN
+F 0 "#PWR012" H 4550 3850 50  0001 C CNN
 F 1 "VCC" V 4550 4200 50  0000 C CNN
 F 2 "" H 4550 4000 50  0001 C CNN
@@
 $EndComp
 $Comp
-L GND #PWR014
+L GND #PWR013
 U 1 1 598F03E6
 P 4800 5250
-F 0 "#PWR014" H 4800 5000 50  0001 C CNN
+F 0 "#PWR013" H 4800 5000 50  0001 C CNN
 F 1 "GND" V 4800 5050 50  0000 C CNN
 F 2 "" H 4800 5250 50  0001 C CNN
@@
 $EndComp
 $Comp
-L GND #PWR015
+L GND #PWR014
 U 1 1 598F1B59
 P 6200 2550
-F 0 "#PWR015" H 6200 2300 50  0001 C CNN
+F 0 "#PWR014" H 6200 2300 50  0001 C CNN
 F 1 "GND" V 6200 2350 50  0000 C CNN
 F 2 "" H 6200 2550 50  0001 C CNN
@@
 $EndComp
 $Comp
-L VCC #PWR016
+L VCC #PWR015
 U 1 1 598F1BAC
 P 6200 2250
-F 0 "#PWR016" H 6200 2100 50  0001 C CNN
+F 0 "#PWR015" H 6200 2100 50  0001 C CNN
 F 1 "VCC" V 6200 2450 50  0000 C CNN
 F 2 "" H 6200 2250 50  0001 C CNN
@@
 $EndComp
 $Comp
-L GND #PWR017
+L GND #PWR016
 U 1 1 598F641F
 P 850 5350
-F 0 "#PWR017" H 850 5100 50  0001 C CNN
+F 0 "#PWR016" H 850 5100 50  0001 C CNN
 F 1 "GND" V 850 5150 50  0000 C CNN
 F 2 "" H 850 5350 50  0001 C CNN
@@
 SW1
 $Comp
-L VCC #PWR018
+L VCC #PWR017
 U 1 1 598F657A
 P 1750 5300
-F 0 "#PWR018" H 1750 5150 50  0001 C CNN
+F 0 "#PWR017" H 1750 5150 50  0001 C CNN
 F 1 "VCC" V 1750 5500 50  0000 C CNN
 F 2 "" H 1750 5300 50  0001 C CNN
@@
 $EndComp
 $Comp
-L GND #PWR019
+L GND #PWR018
 U 1 1 598F6A62
 P 2550 6750
-F 0 "#PWR019" H 2550 6500 50  0001 C CNN
+F 0 "#PWR018" H 2550 6500 50  0001 C CNN
 F 1 "GND" V 2550 6550 50  0000 C CNN
 F 2 "" H 2550 6750 50  0001 C CNN
@@
 SW2
 $Comp
-L VCC #PWR020
+L VCC #PWR019
 U 1 1 598F6A69
 P 1650 6650
-F 0 "#PWR020" H 1650 6500 50  0001 C CNN
+F 0 "#PWR019" H 1650 6500 50  0001 C CNN
 F 1 "VCC" V 1650 6850 50  0000 C CNN
 F 2 "" H 1650 6650 50  0001 C CNN
@@
 NoConn ~ 9050 6000
 $Comp
-L GND #PWR021
-U 1 1 598FA964
-P 9050 5700
-F 0 "#PWR021" H 9050 5450 50  0001 C CNN
-F 1 "GND" V 9050 5500 50  0000 C CNN
-F 2 "" H 9050 5700 50  0001 C CNN
-F 3 "" H 9050 5700 50  0001 C CNN
-	1    9050 5700
-	0    1    1    0
-$EndComp
-$Comp
-L GND #PWR022
+L GND #PWR020
 U 1 1 598FA9CD
 P 9050 4500
-F 0 "#PWR022" H 9050 4250 50  0001 C CNN
+F 0 "#PWR020" H 9050 4250 50  0001 C CNN
 F 1 "GND" V 9050 4300 50  0000 C CNN
 F 2 "" H 9050 4500 50  0001 C CNN
@@
 $EndComp
 $Comp
-L VCC #PWR023
+L VCC #PWR021
 U 1 1 598FAE5F
 P 6800 5600
-F 0 "#PWR023" H 6800 5450 50  0001 C CNN
+F 0 "#PWR021" H 6800 5450 50  0001 C CNN
 F 1 "VCC" V 6800 5800 50  0000 C CNN
 F 2 "" H 6800 5600 50  0001 C CNN
@@
 $EndComp
 $Comp
-L GND #PWR024
-U 1 1 598FB20B
-P 6800 5100
-F 0 "#PWR024" H 6800 4850 50  0001 C CNN
-F 1 "GND" V 6800 4900 50  0000 C CNN
-F 2 "" H 6800 5100 50  0001 C CNN
-F 3 "" H 6800 5100 50  0001 C CNN
-	1    6800 5100
-	0    1    1    0
-$EndComp
-$Comp
-L VCC #PWR025
+L VCC #PWR023
 U 1 1 598FC725
 P 5550 2650
-F 0 "#PWR025" H 5550 2500 50  0001 C CNN
+F 0 "#PWR023" H 5550 2500 50  0001 C CNN
 F 1 "VCC" V 5550 2850 50  0000 C CNN
 F 2 "" H 5550 2650 50  0001 C CNN
@@
 	1    0    0    -1
 $EndComp
+NoConn ~ 9050 5700
+NoConn ~ 6800 4500
+NoConn ~ 6800 5100
 $EndSCHEMATC
