File: KiCadProject/v1.56/PongClock.kicad_pcb (KiCad board)
At the start: 2 copper layers, 67.3 x 88.9 mm, 24 parts, among them J1 CONN_01X01_MALE, J2 MY_USB_OTG, SW1 SW_DIP_x01, SW2 SW_DIP_x01, U1 TinyRTC_I2C_RIGHT, U2 MAX7219_IN, U3 MAX7219_IN, U4 MAX7219_IN, U5 MAX7219_IN, U6 MAX7219_IN, U7 MAX7219_IN, U8 ATMEGA328P-PU, U9 FTDI1232, Y1 Crystal

Commit message: v1.56
Routing:
- net VCC: track 292.6 -> 291.8 mm
- net GND: track 213.9 -> 213.2 mm
Other:
- board text added: "PongClock v1.56"
- board text removed: "PongClock v1.55"
Changed lines of the file:
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@@
     (links 51)
     (no_connects 1)
-    (area 109.144999 46.914999 176.605001 135.965001)
+    (area 82.320001 12.54 218.67 136.36968)
     (thickness 1.6)
     (drawings 22)
-    (tracks 194)
+    (tracks 195)
     (zones 0)
     (modules 24)
@@
     (mod_text_size 1 1)
     (mod_text_width 0.15)
-    (pad_size 1.524 1.524)
-    (pad_drill 0.762)
+    (pad_size 2 2)
+    (pad_drill 1)
     (pad_to_mask_clearance 0.2)
     (aux_axis_origin 106.68 44.45)
@@
     (fp_line (start 3.175 11.43) (end 17.145 11.43) (layer F.CrtYd) (width 0.15))
     (fp_line (start 17.145 -3.81) (end 3.175 -3.81) (layer F.CrtYd) (width 0.15))
-    (pad 5 thru_hole circle (at 5.08 10.16 90) (size 1.524 1.524) (drill 0.762) (layers *.Cu *.Mask)
+    (pad 5 thru_hole oval (at 5.08 10.16 90) (size 2 4) (drill 1) (layers *.Cu *.Mask)
       (net 7 GND))
-    (pad 4 thru_hole circle (at 7.62 10.16 180) (size 1.524 1.524) (drill 0.762) (layers *.Cu *.Mask))
-    (pad 3 thru_hole circle (at 10.16 10.16 90) (size 1.524 1.524) (drill 0.762) (layers *.Cu *.Mask))
-    (pad 2 thru_hole circle (at 12.7 10.16 90) (size 1.524 1.524) (drill 0.762) (layers *.Cu *.Mask))
-    (pad 1 thru_hole circle (at 15.24 10.16 90) (size 1.524 1.524) (drill 0.762) (layers *.Cu *.Mask)
+    (pad 4 thru_hole oval (at 7.62 10.16 90) (size 2 4) (drill 1) (layers *.Cu *.Mask))
+    (pad 3 thru_hole oval (at 10.16 10.16 90) (size 2 4) (drill 1) (layers *.Cu *.Mask))
+    (pad 2 thru_hole oval (at 12.7 10.16 90) (size 2 4) (drill 1) (layers *.Cu *.Mask))
+    (pad 1 thru_hole oval (at 15.24 10.16 90) (size 2 4) (drill 1) (layers *.Cu *.Mask)
       (net 6 VCC))
-    (pad 6 thru_hole circle (at 15.875 2.54 90) (size 1.524 1.524) (drill 0.762) (layers *.Cu *.Mask)
+    (pad 6 thru_hole circle (at 15.875 2.54 90) (size 2 2) (drill 1) (layers *.Cu *.Mask)
       (net 14 "Net-(J2-Pad6)"))
-    (pad 6 thru_hole circle (at 4.445 2.54 90) (size 1.524 1.524) (drill 0.762) (layers *.Cu *.Mask)
+    (pad 6 thru_hole circle (at 4.445 2.54 90) (size 2 2) (drill 1) (layers *.Cu *.Mask)
       (net 14 "Net-(J2-Pad6)"))
   )
@@
     (arrow2b (pts (xy 210.82 119.38) (xy 211.406421 120.506504)))
   )
-  (gr_text "PongClock v1.55" (at 162.56 62.23 90) (layer Eco2.User)
+  (gr_text "PongClock v1.56" (at 162.56 62.23 90) (layer Eco2.User)
     (effects (font (size 1.5 1.5) (thickness 0.3)))
   )
@@
   (segment (start 140.97 92.71) (end 140.97 88.9) (width 1) (layer F.Cu) (net 5))
   (segment (start 140.97 88.9) (end 147.32 82.55) (width 1) (layer F.Cu) (net 5))
-  (segment (start 134.62 111.76) (end 135.89 113.03) (width 1) (layer F.Cu) (net 6))
-  (segment (start 135.89 113.03) (end 140.97 113.03) (width 1) (layer F.Cu) (net 6))
-  (segment (start 134.62 105.41) (end 134.62 111.76) (width 1) (layer B.Cu) (net 6))
-  (via (at 134.62 111.76) (size 2) (drill 1) (layers F.Cu B.Cu) (net 6))
+  (segment (start 135.619999 111.489999) (end 134.62 110.49) (width 1) (layer F.Cu) (net 6))
+  (segment (start 137.16 113.03) (end 135.619999 111.489999) (width 1) (layer F.Cu) (net 6))
+  (segment (start 140.97 113.03) (end 137.16 113.03) (width 1) (layer F.Cu) (net 6))
+  (segment (start 134.62 105.41) (end 134.62 110.49) (width 1) (layer B.Cu) (net 6))
+  (via (at 134.62 110.49) (size 2) (drill 1) (layers F.Cu B.Cu) (net 6))
   (segment (start 124.46 98.425) (end 127.635 98.425) (width 1) (layer F.Cu) (net 6))
   (via (at 134.62 105.41) (size 2) (drill 1) (layers F.Cu B.Cu) (net 6))
@@
   (segment (start 140.477999 80.787999) (end 141.478001 81.788001) (width 1) (layer F.Cu) (net 6))
   (segment (start 141.478001 81.788001) (end 142.24 82.55) (width 1) (layer F.Cu) (net 6))
+  (segment (start 137.16 107.95) (end 140.97 107.95) (width 1) (layer F.Cu) (net 7))
+  (segment (start 124.46 108.585) (end 125.095 107.95) (width 1) (layer F.Cu) (net 7))
+  (segment (start 125.095 107.95) (end 137.16 107.95) (width 1) (layer F.Cu) (net 7))
+  (segment (start 139.7 82.55) (end 137.16 85.09) (width 1) (layer F.Cu) (net 7))
+  (segment (start 137.16 85.09) (end 137.16 86.36) (width 1) (layer F.Cu) (net 7))
+  (segment (start 137.16 86.36) (end 137.16 107.95) (width 1) (layer F.Cu) (net 7))
   (segment (start 163.83 118.11) (end 158.79 118.11) (width 1) (layer F.Cu) (net 7))
   (segment (start 158.79 118.11) (end 158.75 118.07) (width 1) (layer F.Cu) (net 7))
@@
   (segment (start 168.91 110.49) (end 158.79 110.49) (width 1) (layer F.Cu) (net 7))
   (segment (start 158.79 110.49) (end 158.75 110.53) (width 1) (layer F.Cu) (net 7))
-  (segment (start 139.7 82.55) (end 137.16 85.09) (width 1) (layer F.Cu) (net 7))
-  (segment (start 137.16 85.09) (end 137.16 86.36) (width 1) (layer F.Cu) (net 7))
-  (segment (start 137.16 86.36) (end 137.16 108.585) (width 1) (layer F.Cu) (net 7))
   (segment (start 115.57 90.17) (end 111.76 90.17) (width 1) (layer F.Cu) (net 7))
   (segment (start 115.57 95.25) (end 115.57 90.17) (width 1) (layer B.Cu) (net 7))
@@
   (segment (start 111.76 118.11) (end 114.935 118.11) (width 1) (layer F.Cu) (net 7))
   (segment (start 114.935 118.11) (end 124.46 108.585) (width 1) (layer F.Cu) (net 7))
-  (segment (start 124.46 108.585) (end 137.16 108.585) (width 1) (layer F.Cu) (net 7))
-  (segment (start 137.16 108.585) (end 140.335 108.585) (width 1) (layer F.Cu) (net 7))
-  (segment (start 140.335 108.585) (end 140.97 107.95) (width 1) (layer F.Cu) (net 7))
   (segment (start 158.75 110.53) (end 148.63 110.53) (width 1) (layer F.Cu) (net 7))
   (segment (start 148.63 110.53) (end 148.59 110.49) (width 1) (layer F.Cu) (net 7))
