File: KiCadProject/v1.57/PongClock.kicad_pcb (KiCad board)
At the start: 2 copper layers, 67.3 x 88.9 mm, 24 parts, among them J1 CONN_01X01_MALE, J2 MY_USB_OTG, SW1 SW_DIP_x01, SW2 SW_DIP_x01, U1 TinyRTC_I2C_RIGHT, U2 MAX7219_IN, U3 MAX7219_IN, U4 MAX7219_IN, U5 MAX7219_IN, U6 MAX7219_IN, U7 MAX7219_IN, U8 ATMEGA328P-PU, U9 FTDI1232, Y1 Crystal

Commit message: v1.57
Parts:
- added R5: 10k, Resistors_SMD:R_1206_HandSoldering, F.Cu at (137.2, 99.8)
- added R6: R_PHOTO, PongClock:MY_PHOTO_RESITOR, F.Cu at (127.0, 127.0)
- C3: footprint Capacitors_THT:CP_Radial_D5.0mm_P2.50mm -> Capacitors_SMD:C_1206_HandSoldering; moved to F.Cu
- moved SW2 82.8 mm to (120.7, 49.5)
- moved SW1 82.7 mm to (165.1, 49.5), turned to 180 degrees
- moved C5 75.1 mm to (122.5, 53.3)
- moved C4 75.0 mm to (163.3, 53.3), turned to 0 degrees
- moved R1 20.5 mm to (156.9, 105.4)
- moved R2 7.73 mm to (126.3, 118.1)
- moved C3 2.00 mm to (154.4, 92.7)
Connections:
- J2 pad 6: Net-(J2-Pad6) -> (no net)
- U8 pad 11: MAX_IN -> LATCH
- U8 pad 12: LATCH -> CLK
- U8 pad 13: CLK -> MAX_IN
- U8 pad 26: (no net) -> PHOTO
Routing:
- net SW2: track 59.9 -> 147.4 mm, vias 2 -> 4
- net PHOTO: track 0.00 -> 41.6 mm, vias 0 -> 2
- net SW1: track 40.9 -> 75.0 mm
- net VCC: track 291.8 -> 281.6 mm
- net MAX_IN: track 31.6 -> 21.5 mm, vias 2 -> 0
- net LATCH: track 107.6 -> 112.5 mm
- net CLK: track 101.3 -> 99.7 mm
- net DTR: track 16.1 -> 14.6 mm
- net GND: track 213.2 -> 212.1 mm
- added copper zone on F.Cu, net GND
Other:
- board size 67.3 x 88.9 mm -> 67.3 x 90.2 mm
- net class 0,4mm removed
- board text added: "PongClock v1.57"
- board text removed: "PongClock v1.56"
