File: KiCadProject/v1.57/PongClock_rotate.kicad_pcb (KiCad board)
At the start: 2 copper layers, 88.9 x 67.3 mm, 24 parts, among them J1 CONN_01X01_MALE, J2 MY_USB_OTG, SW1 SW_DIP_x01, SW2 SW_DIP_x01, U1 TinyRTC_I2C_RIGHT, U2 MAX7219_IN, U3 MAX7219_IN, U4 MAX7219_IN, U5 MAX7219_IN, U6 MAX7219_IN, U7 MAX7219_IN, U8 ATMEGA328P-PU, U9 FTDI1232, Y1 Crystal

Commit message: v1.57
Parts:
- added R5: 10k, Resistors_SMD:R_1206_HandSoldering, F.Cu at (172.2, 88.9)
- added R6: R_PHOTO, PongClock:MY_PHOTO_RESITOR, F.Cu at (199.4, 99.1)
- C3: footprint Capacitors_THT:CP_Radial_D5.0mm_P2.50mm -> Capacitors_SMD:C_1206_HandSoldering; moved to F.Cu
- moved SW1 65.1 mm to (121.9, 61.0), turned to 270 degrees
- moved SW2 65.0 mm to (121.9, 105.4)
- moved C4 57.4 mm to (125.7, 62.8), turned to 90 degrees
- moved C5 57.3 mm to (125.7, 103.6)
- moved C3 18.1 mm to (165.1, 71.6)
- moved C1 17.8 mm to (185.4, 67.3)
- moved C2 17.8 mm to (188.0, 67.3)
- moved D1 17.8 mm to (179.8, 81.3)
- moved J1 17.8 mm to (204.5, 59.7)
- moved J2 17.8 mm to (186.1, 111.8)
- moved R3 17.8 mm to (173.9, 81.3)
- moved R4 17.8 mm to (160.0, 71.7)
- moved U1 17.8 mm to (134.6, 81.3)
- moved U2 17.8 mm to (121.9, 114.3)
- moved U3 17.8 mm to (165.1, 114.3)
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Connections:
- J2 pad 6: Net-(J2-Pad6) -> (no net)
- U8 pad 11: MAX_IN -> LATCH
- U8 pad 12: LATCH -> CLK
- U8 pad 13: CLK -> MAX_IN
- U8 pad 26: (no net) -> PHOTO
Routing:
- net SW2: track 59.9 -> 147.4 mm, vias 2 -> 4
- net PHOTO: track 0.00 -> 41.6 mm, vias 0 -> 2
- net SW1: track 40.9 -> 75.0 mm
- net VCC: track 291.8 -> 281.6 mm
- net MAX_IN: track 31.6 -> 21.5 mm, vias 2 -> 0
- net LATCH: track 107.6 -> 112.5 mm
- net CLK: track 101.3 -> 99.7 mm
- net DTR: track 16.1 -> 14.6 mm
- net GND: track 213.2 -> 212.1 mm
- added copper zone on F.Cu, net GND
Other:
- board size 88.9 x 67.3 mm -> 90.2 x 67.3 mm
- net class 0,4mm removed
- board text added: "PongClock v1.57"
- board text removed: "PongClock v1.56"
