File: KiCadProject/v1.57/PongClock.sch (KiCad schematic (older format))
At the start: 26 parts, among them J1 CONN_01X01_MALE, J2 MY_USB_OTG, SW1 SW_DIP_x01, SW2 SW_DIP_x01, U1 TinyRTC_I2C_RIGHT, U2 MAX7219_IN, U3 MAX7219_IN, U4 MAX7219_IN, U5 MAX7219_IN, U6 MAX7219_IN, U7 MAX7219_IN, U8 ATMEGA328P-PU, U9 FTDI1232, Y1 Crystal

Commit message: v1.58
Parts:
- R6: footprint (none) -> PongClock:MY_PHOTO_RESITOR
Changed lines of the file:
@@
 $EndComp
 $Comp
-L VCC #PWR14
+L VCC #PWR01
 U 1 1 596A2EB4
 P 6800 4400
-F 0 "#PWR14" H 6800 4250 50  0001 C CNN
+F 0 "#PWR01" H 6800 4250 50  0001 C CNN
 F 1 "VCC" V 6800 4600 50  0000 C CNN
 F 2 "" H 6800 4400 50  0001 C CNN
@@
 $EndComp
 $Comp
-L GND #PWR23
+L GND #PWR02
 U 1 1 597B8E84
 P 6800 5700
-F 0 "#PWR23" H 6800 5450 50  0001 C CNN
+F 0 "#PWR02" H 6800 5450 50  0001 C CNN
 F 1 "GND" V 6800 5500 50  0000 C CNN
 F 2 "" H 6800 5700 50  0001 C CNN
@@
 NoConn ~ 6800 4800
 $Comp
-L VCC #PWR18
+L VCC #PWR03
 U 1 1 597C7538
 P 6800 5000
-F 0 "#PWR18" H 6800 4850 50  0001 C CNN
+F 0 "#PWR03" H 6800 4850 50  0001 C CNN
 F 1 "VCC" V 6800 5200 50  0000 C CNN
 F 2 "" H 6800 5000 50  0001 C CNN
@@
 $EndComp
 $Comp
-L GND #PWR8
+L GND #PWR04
 U 1 1 598DFC0D
 P 1050 3300
-F 0 "#PWR8" H 1050 3050 50  0001 C CNN
+F 0 "#PWR04" H 1050 3050 50  0001 C CNN
 F 1 "GND" V 1050 3100 50  0000 C CNN
 F 2 "" H 1050 3300 50  0001 C CNN
@@
 $EndComp
 $Comp
-L VCC #PWR1
+L VCC #PWR05
 U 1 1 598DFC7E
 P 1050 1350
-F 0 "#PWR1" H 1050 1200 50  0001 C CNN
+F 0 "#PWR05" H 1050 1200 50  0001 C CNN
 F 1 "VCC" V 1050 1550 50  0000 C CNN
 F 2 "" H 1050 1350 50  0001 C CNN
@@
 OSC1
 $Comp
-L GND #PWR3
+L GND #PWR06
 U 1 1 598E0208
 P 4300 1500
-F 0 "#PWR3" H 4300 1250 50  0001 C CNN
+F 0 "#PWR06" H 4300 1250 50  0001 C CNN
 F 1 "GND" V 4300 1300 50  0000 C CNN
 F 2 "" H 4300 1500 50  0001 C CNN
@@
 $EndComp
 $Comp
-L GND #PWR7
+L GND #PWR07
 U 1 1 598E32E5
 P 4150 3050
-F 0 "#PWR7" H 4150 2800 50  0001 C CNN
+F 0 "#PWR07" H 4150 2800 50  0001 C CNN
 F 1 "GND" V 4150 2850 50  0000 C CNN
 F 2 "" H 4150 3050 50  0001 C CNN
@@
 $EndComp
 $Comp
-L VCC #PWR6
+L VCC #PWR08
 U 1 1 598E33DE
 P 4150 2750
-F 0 "#PWR6" H 4150 2600 50  0001 C CNN
+F 0 "#PWR08" H 4150 2600 50  0001 C CNN
 F 1 "VCC" V 4150 2950 50  0000 C CNN
 F 2 "" H 4150 2750 50  0001 C CNN
@@
 SW2
 $Comp
-L GND #PWR16
+L GND #PWR09
 U 1 1 598EBAEB
 P 4250 4600
-F 0 "#PWR16" H 4250 4350 50  0001 C CNN
+F 0 "#PWR09" H 4250 4350 50  0001 C CNN
 F 1 "GND" V 4250 4400 50  0000 C CNN
 F 2 "" H 4250 4600 50  0001 C CNN
@@
 $EndComp
 $Comp
-L VCC #PWR9
+L VCC #PWR010
 U 1 1 598EBB74
 P 4550 4000
-F 0 "#PWR9" H 4550 3850 50  0001 C CNN
+F 0 "#PWR010" H 4550 3850 50  0001 C CNN
 F 1 "VCC" V 4550 4200 50  0000 C CNN
 F 2 "" H 4550 4000 50  0001 C CNN
@@
 $EndComp
 $Comp
-L GND #PWR17
+L GND #PWR011
 U 1 1 598F03E6
 P 1750 4950
-F 0 "#PWR17" H 1750 4700 50  0001 C CNN
+F 0 "#PWR011" H 1750 4700 50  0001 C CNN
 F 1 "GND" V 1750 4750 50  0000 C CNN
 F 2 "" H 1750 4950 50  0001 C CNN
@@
 $EndComp
 $Comp
-L GND #PWR4
+L GND #PWR012
 U 1 1 598F1B59
 P 5650 1650
-F 0 "#PWR4" H 5650 1400 50  0001 C CNN
+F 0 "#PWR012" H 5650 1400 50  0001 C CNN
 F 1 "GND" V 5650 1450 50  0000 C CNN
 F 2 "" H 5650 1650 50  0001 C CNN
@@
 $EndComp
 $Comp
-L VCC #PWR2
+L VCC #PWR013
 U 1 1 598F1BAC
 P 5650 1350
-F 0 "#PWR2" H 5650 1200 50  0001 C CNN
+F 0 "#PWR013" H 5650 1200 50  0001 C CNN
 F 1 "VCC" V 5650 1550 50  0000 C CNN
 F 2 "" H 5650 1350 50  0001 C CNN
@@
 $EndComp
 $Comp
-L GND #PWR12
+L GND #PWR014
 U 1 1 598F641F
 P 1000 4250
-F 0 "#PWR12" H 1000 4000 50  0001 C CNN
+F 0 "#PWR014" H 1000 4000 50  0001 C CNN
 F 1 "GND" V 1000 4050 50  0000 C CNN
 F 2 "" H 1000 4250 50  0001 C CNN
@@
 SW1
 $Comp
-L VCC #PWR10
+L VCC #PWR015
 U 1 1 598F657A
 P 1900 4200
-F 0 "#PWR10" H 1900 4050 50  0001 C CNN
+F 0 "#PWR015" H 1900 4050 50  0001 C CNN
 F 1 "VCC" V 1900 4400 50  0000 C CNN
 F 2 "" H 1900 4200 50  0001 C CNN
@@
 $EndComp
 $Comp
-L GND #PWR13
+L GND #PWR016
 U 1 1 598F6A62
 P 3400 4300
-F 0 "#PWR13" H 3400 4050 50  0001 C CNN
+F 0 "#PWR016" H 3400 4050 50  0001 C CNN
 F 1 "GND" V 3400 4100 50  0000 C CNN
 F 2 "" H 3400 4300 50  0001 C CNN
@@
 SW2
 $Comp
-L VCC #PWR11
+L VCC #PWR017
 U 1 1 598F6A69
 P 2500 4200
-F 0 "#PWR11" H 2500 4050 50  0001 C CNN
+F 0 "#PWR017" H 2500 4050 50  0001 C CNN
 F 1 "VCC" V 2500 4400 50  0000 C CNN
 F 2 "" H 2500 4200 50  0001 C CNN
@@
 Connection ~ 1900 4200
 $Comp
-L VCC #PWR22
+L VCC #PWR018
 U 1 1 598FAE5F
 P 6800 5600
-F 0 "#PWR22" H 6800 5450 50  0001 C CNN
+F 0 "#PWR018" H 6800 5450 50  0001 C CNN
 F 1 "VCC" V 6800 5800 50  0000 C CNN
 F 2 "" H 6800 5600 50  0001 C CNN
@@
 $EndComp
 $Comp
-L VCC #PWR5
+L VCC #PWR019
 U 1 1 598FC725
 P 5900 2650
-F 0 "#PWR5" H 5900 2500 50  0001 C CNN
+F 0 "#PWR019" H 5900 2500 50  0001 C CNN
 F 1 "VCC" V 5900 2850 50  0000 C CNN
 F 2 "" H 5900 2650 50  0001 C CNN
@@
 LATCH
 $Comp
-L GND #PWR19
+L GND #PWR020
 U 1 1 59935016
 P 6800 5100
-F 0 "#PWR19" H 6800 4850 50  0001 C CNN
+F 0 "#PWR020" H 6800 4850 50  0001 C CNN
 F 1 "GND" V 6800 4900 50  0000 C CNN
 F 2 "" H 6800 5100 50  0001 C CNN
@@
 $EndComp
 $Comp
-L GND #PWR15
+L GND #PWR021
 U 1 1 59935069
 P 6800 4500
-F 0 "#PWR15" H 6800 4250 50  0001 C CNN
+F 0 "#PWR021" H 6800 4250 50  0001 C CNN
 F 1 "GND" V 6800 4300 50  0000 C CNN
 F 2 "" H 6800 4500 50  0001 C CNN
@@
 F 0 "R6" H 1950 5650 50  0000 L CNN
 F 1 "R_PHOTO" H 1950 5600 50  0000 L TNN
-F 2 "" V 1950 5350 50  0001 L CNN
+F 2 "PongClock:MY_PHOTO_RESITOR" V 1950 5350 50  0001 L CNN
 F 3 "" H 1900 5550 50  0001 C CNN
 	1    1900 5600
@@
 $EndComp
 $Comp
-L VCC #PWR21
+L VCC #PWR022
 U 1 1 5999D7E2
 P 2050 5600
-F 0 "#PWR21" H 2050 5450 50  0001 C CNN
+F 0 "#PWR022" H 2050 5450 50  0001 C CNN
 F 1 "VCC" V 2050 5800 50  0000 C CNN
 F 2 "" H 2050 5600 50  0001 C CNN
@@
 $EndComp
 $Comp
-L GND #PWR20
+L GND #PWR023
 U 1 1 5999D8E6
 P 1450 5600
-F 0 "#PWR20" H 1450 5350 50  0001 C CNN
+F 0 "#PWR023" H 1450 5350 50  0001 C CNN
 F 1 "GND" V 1450 5400 50  0000 C CNN
 F 2 "" H 1450 5600 50  0001 C CNN
