File: KiCadProject/v1.60/PongClock.kicad_pcb (KiCad board)
At the start: 2 copper layers, 67.3 x 90.2 mm, 29 parts, among them J1 CONN_01X01_MALE, J2 MY_USB_OTG, SW1 SW_DIP_x01, SW2 SW_DIP_x01, U1 TinyRTC_I2C_RIGHT, U2 MAX7219_IN, U3 MAX7219_IN, U4 MAX7219_IN, U5 MAX7219_IN, U6 MAX7219_IN, U7 MAX7219_IN, U8 ATMEGA328P-PU, U9 FTDI1232, Y1 Crystal

Commit message: v1.60
Parts:
- R3: footprint Resistors_SMD:R_0805_HandSoldering -> Resistors_SMD:R_1206_HandSoldering
- SW1, SW2: footprint mod_switch:smd_push -> PongClock:MEDIUM_BUTTON
- moved C4 10.2 mm to (164.5, 63.5)
- moved C5 10.2 mm to (121.3, 63.5)
- moved SW2 5.75 mm to (121.3, 55.2)
- moved SW1 5.73 mm to (164.5, 55.2)
- moved D1 1.17 mm to (144.8, 108.6)
- moved R3 0.72 mm to (144.8, 102.2)
Routing:
- net VCC: track 287.4 -> 272.8 mm
- net SW1: track 67.1 -> 56.8 mm
- net SW2: track 147.4 -> 138.2 mm
Other:
- board text added: "PongClock v1.60"
- board text removed: "PongClock v1.59"
