File: KiCadProject/v1.60/PongClock.sch (KiCad schematic (older format))
At the start: 29 parts, among them J1 CONN_01X01_MALE, J2 MY_USB_OTG, SW1 SW_DIP_x01, SW2 SW_DIP_x01, U1 TinyRTC_I2C_RIGHT, U2 MAX7219_IN, U3 MAX7219_IN, U4 MAX7219_IN, U5 MAX7219_IN, U6 MAX7219_IN, U7 MAX7219_IN, U8 ATMEGA328P-PU, U9 FTDI1232, Y1 Crystal

Commit message: v1.60
Parts:
- R3: footprint Resistors_SMD:R_0805_HandSoldering -> Resistors_SMD:R_1206_HandSoldering
- SW1, SW2: footprint mod_switch:smd_push -> PongClock:MEDIUM_BUTTON
Other:
- note added: "LED"
- note added: "Light Sensor"
- moved on the sheet: D1, R3, R5, R6
Changed lines of the file:
@@
 Text GLabel 3250 2850 2    60   Input ~ 0
 LED
-Text GLabel 1150 4950 0    60   Input ~ 0
+Text GLabel 2550 5700 0    60   Input ~ 0
 LED
 $Comp
 L R R3
 U 1 1 598EFE16
-P 1300 4950
-F 0 "R3" V 1380 4950 50  0000 C CNN
-F 1 "R_LED" V 1200 4950 50  0000 C CNN
-F 2 "Resistors_SMD:R_0805_HandSoldering" V 1230 4950 50  0001 C CNN
-F 3 "" H 1300 4950 50  0001 C CNN
-	1    1300 4950
+P 2700 5700
+F 0 "R3" V 2780 5700 50  0000 C CNN
+F 1 "R_LED" V 2600 5700 50  0000 C CNN
+F 2 "Resistors_SMD:R_1206_HandSoldering" V 2630 5700 50  0001 C CNN
+F 3 "" H 2700 5700 50  0001 C CNN
+	1    2700 5700
 	0    1    1    0
 $EndComp
@@
 L LED D1
 U 1 1 598F0345
-P 1600 4950
-F 0 "D1" H 1600 5050 50  0000 C CNN
-F 1 "LED" H 1600 4850 50  0000 C CNN
-F 2 "LEDs:LED_1206_HandSoldering" H 1600 4950 50  0001 C CNN
-F 3 "" H 1600 4950 50  0001 C CNN
-	1    1600 4950
+P 3000 5700
+F 0 "D1" H 3000 5800 50  0000 C CNN
+F 1 "LED" H 3000 5600 50  0000 C CNN
+F 2 "LEDs:LED_1206_HandSoldering" H 3000 5700 50  0001 C CNN
+F 3 "" H 3000 5700 50  0001 C CNN
+	1    3000 5700
 	-1   0    0    1
 $EndComp
@@
 L GND #PWR010
 U 1 1 598F03E6
-P 1750 4950
-F 0 "#PWR010" H 1750 4700 50  0001 C CNN
-F 1 "GND" V 1750 4750 50  0000 C CNN
-F 2 "" H 1750 4950 50  0001 C CNN
-F 3 "" H 1750 4950 50  0001 C CNN
-	1    1750 4950
+P 3150 5700
+F 0 "#PWR010" H 3150 5450 50  0001 C CNN
+F 1 "GND" V 3150 5500 50  0000 C CNN
+F 2 "" H 3150 5700 50  0001 C CNN
+F 3 "" H 3150 5700 50  0001 C CNN
+	1    3150 5700
 	0    -1   -1   0
 $EndComp
@@
 F 0 "SW1" H 1600 4500 50  0000 C CNN
 F 1 "SW_DIP_x01" H 1600 4200 50  0000 C CNN
-F 2 "mod_switch:smd_push" H 1600 4350 50  0001 C CNN
+F 2 "PongClock:MEDIUM_BUTTON" H 1600 4350 50  0001 C CNN
 F 3 "" H 1600 4350 50  0001 C CNN
 	1    1600 4350
@@
 F 0 "SW2" H 2800 4500 50  0000 C CNN
 F 1 "SW_DIP_x01" H 2800 4200 50  0000 C CNN
-F 2 "mod_switch:smd_push" H 2800 4350 50  0001 C CNN
+F 2 "PongClock:MEDIUM_BUTTON" H 2800 4350 50  0001 C CNN
 F 3 "" H 2800 4350 50  0001 C CNN
 	1    2800 4350
@@
 L R_PHOTO R6
 U 1 1 5999D738
-P 1900 5600
-F 0 "R6" H 1950 5650 50  0000 L CNN
-F 1 "R_PHOTO" H 1950 5600 50  0000 L TNN
-F 2 "PongClock:MY_PHOTO_RESITOR" V 1950 5350 50  0001 L CNN
-F 3 "" H 1900 5550 50  0001 C CNN
-	1    1900 5600
+P 1750 5700
+F 0 "R6" H 1800 5750 50  0000 L CNN
+F 1 "R_PHOTO" H 1800 5700 50  0000 L TNN
+F 2 "PongClock:MY_PHOTO_RESITOR" V 1800 5450 50  0001 L CNN
+F 3 "" H 1750 5650 50  0001 C CNN
+	1    1750 5700
 	0    1    1    0
 $EndComp
@@
 L VCC #PWR021
 U 1 1 5999D7E2
-P 2050 5600
-F 0 "#PWR021" H 2050 5450 50  0001 C CNN
-F 1 "VCC" V 2050 5800 50  0000 C CNN
-F 2 "" H 2050 5600 50  0001 C CNN
-F 3 "" H 2050 5600 50  0001 C CNN
-	1    2050 5600
+P 1900 5700
+F 0 "#PWR021" H 1900 5550 50  0001 C CNN
+F 1 "VCC" V 1900 5900 50  0000 C CNN
+F 2 "" H 1900 5700 50  0001 C CNN
+F 3 "" H 1900 5700 50  0001 C CNN
+	1    1900 5700
 	0    1    1    0
 $EndComp
@@
 L R R5
 U 1 1 5999D838
-P 1600 5600
-F 0 "R5" V 1680 5600 50  0000 C CNN
-F 1 "10k" V 1600 5600 50  0000 C CNN
-F 2 "Resistors_SMD:R_1206_HandSoldering" V 1530 5600 50  0001 C CNN
-F 3 "" H 1600 5600 50  0001 C CNN
-	1    1600 5600
+P 1450 5700
+F 0 "R5" V 1530 5700 50  0000 C CNN
+F 1 "10k" V 1450 5700 50  0000 C CNN
+F 2 "Resistors_SMD:R_1206_HandSoldering" V 1380 5700 50  0001 C CNN
+F 3 "" H 1450 5700 50  0001 C CNN
+	1    1450 5700
 	0    -1   -1   0
 $EndComp
@@
 L GND #PWR022
 U 1 1 5999D8E6
-P 1450 5600
-F 0 "#PWR022" H 1450 5350 50  0001 C CNN
-F 1 "GND" V 1450 5400 50  0000 C CNN
-F 2 "" H 1450 5600 50  0001 C CNN
-F 3 "" H 1450 5600 50  0001 C CNN
-	1    1450 5600
-	0    1    1    0
-$EndComp
-Text GLabel 1750 5600 1    60   Input ~ 0
+P 1300 5700
+F 0 "#PWR022" H 1300 5450 50  0001 C CNN
+F 1 "GND" V 1300 5500 50  0000 C CNN
+F 2 "" H 1300 5700 50  0001 C CNN
+F 3 "" H 1300 5700 50  0001 C CNN
+	1    1300 5700
+	0    1    1    0
+$EndComp
+Text GLabel 1600 5700 1    60   Input ~ 0
 PHOTO
 Text GLabel 3250 2200 2    60   Input ~ 0
@@
 	0    1    1    0
 $EndComp
+Text Notes 1350 5200 0    60   ~ 0
+Light Sensor
+Text Notes 2650 5200 0    60   ~ 0
+LED
+Wire Notes Line
+	2000 5150 2200 5150
+Wire Notes Line
+	2200 5150 2200 6200
+Wire Notes Line
+	2200 6200 950  6200
+Wire Notes Line
+	950  6200 950  5150
+Wire Notes Line
+	950  5150 1300 5150
 $EndSCHEMATC
