File: KiCadProject/v1.60/PongClock_rotate.kicad_pcb (KiCad board)
At the start: 2 copper layers, 90.2 x 67.3 mm, 29 parts, among them J1 CONN_01X01_MALE, J2 MY_USB_OTG, SW1 SW_DIP_x01, SW2 SW_DIP_x01, U1 TinyRTC_I2C_RIGHT, U2 MAX7219_IN, U3 MAX7219_IN, U4 MAX7219_IN, U5 MAX7219_IN, U6 MAX7219_IN, U7 MAX7219_IN, U8 ATMEGA328P-PU, U9 FTDI1232, Y1 Crystal

Commit message: v1.60
Parts:
- R3: footprint Resistors_SMD:R_0805_HandSoldering -> Resistors_SMD:R_1206_HandSoldering
- SW1, SW2: footprint mod_switch:smd_push -> PongClock:MEDIUM_BUTTON
- moved C5 10.6 mm to (123.5, 99.9)
- moved C4 10.6 mm to (123.5, 56.7)
- moved SW1 6.09 mm to (115.3, 56.7)
- moved SW2 6.08 mm to (115.3, 99.9)
- moved D1 1.53 mm to (168.6, 76.4)
- moved R3 1.07 mm to (162.3, 76.4)
- moved C7 0.38 mm to (168.0, 66.8)
- moved R5 0.38 mm to (159.8, 84.0)
- moved C2 0.38 mm to (175.6, 61.7)
- moved R1 0.38 mm to (165.4, 61.7)
- moved U9 0.38 mm to (157.8, 52.2)
- moved J2 0.38 mm to (173.7, 106.8)
- moved R4 0.38 mm to (147.7, 66.7)
- moved R7 0.38 mm to (133.7, 55.5)
- moved U4 0.38 mm to (175.6, 109.4)
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Routing:
- net VCC: track 287.4 -> 272.8 mm
- net SW1: track 67.1 -> 56.8 mm
- net SW2: track 147.4 -> 138.2 mm
Other:
- board text added: "PongClock v1.60"
- board text removed: "PongClock v1.59"
